Commit message: added some parameters

File: urdf/simple_arm.xacro (robot description, xacro)
@@ -1,3 +1,10 @@
-<robot name="test_robot">
+<?xml version="1.0"?>
+<robot xmlns:xacro="oarkit" name="test_robot">
+  <xacro:property name="pi" value="3.1415926535897931" />
+  <xacro:property name="xl320_height" value=".024" />
+  <xacro:property name="xl320_length" value=".036" />
+  <xacro:property name="xl320_width" value=".027" />
+  <xacro:property name="link1_length" value=".2" />
+  <xacro:property name="link2_length" value=".2" />
   <link name="link1" />
   <link name="link2" />
@@ -8,8 +15,10 @@
     <parent link="link1"/>
     <child link="link2"/>
+    <origin xyz="0 0 0" rpy="0 0 0" />
   </joint>
   <joint name="joint2" type="continuous">
     <parent link="link2"/>
     <child link="link3"/>
+    <origin xyz="0 0 0" rpy="0 0 0" />
   </joint>
   <joint name="joint3" type="continuous">

Commit message: updated basic robot shape

File: urdf/simple_arm.xacro (robot description, xacro)
@@ -1,4 +1,4 @@
 <?xml version="1.0"?>
-<robot xmlns:xacro="oarkit" name="test_robot">
+<robot xmlns:xacro="http://www.ros.org/wiki/xacro" name="test_robot">
   <xacro:property name="pi" value="3.1415926535897931" />
   <xacro:property name="xl320_height" value=".024" />
@@ -15,18 +15,20 @@
     <parent link="link1"/>
     <child link="link2"/>
-    <origin xyz="0 0 0" rpy="0 0 0" />
+    <origin xyz="0 0 0" rpy="0 -${pi/2} 0" />
   </joint>
   <joint name="joint2" type="continuous">
     <parent link="link2"/>
     <child link="link3"/>
-    <origin xyz="0 0 0" rpy="0 0 0" />
+    <origin xyz="${xl320_width} 0 0" rpy="0 0 ${-pi/2}" />
   </joint>
   <joint name="joint3" type="continuous">
     <parent link="link3"/>
     <child link="link4"/>
+    <origin xyz="0 ${link1_length} 0" rpy="0 0 0" />
   </joint>
   <joint name="joint4" type="continuous">
     <parent link="link4"/>
     <child link="link5"/>
+    <origin xyz="0 ${link1_length} 0" rpy="0 0 0" />
   </joint>
 </robot>

Commit message: added launch files and gave the arm a dummy end effector

File: urdf/simple_arm.xacro (robot description, xacro)
@@ -7,4 +7,5 @@
   <xacro:property name="link1_length" value=".2" />
   <xacro:property name="link2_length" value=".2" />
+  <xacro:property name="end_effector_length" value=".05" />
   <link name="link1" />
   <link name="link2" />
@@ -12,4 +13,6 @@
   <link name="link4" />
   <link name="link5" />
+  <link name="link6" />
+  <link name="link7" />
   <joint name="joint1" type="continuous">
     <parent link="link1"/>
@@ -32,3 +35,13 @@
     <origin xyz="0 ${link1_length} 0" rpy="0 0 0" />
   </joint>
+  <joint name="joint5" type="continuous">
+    <parent link="link5"/>
+    <child link="link6"/>
+    <origin xyz="0 ${xl320_width} 0" rpy="0 0 ${pi/2}" />
+  </joint>
+  <joint name="joint6" type="fixed">
+    <parent link="link6"/>
+    <child link="link7"/>
+    <origin xyz="${end_effector_length} 0 0" rpy="0 0 0" />
+  </joint>
 </robot>
